File: hw/uTrakHF.sch (EAGLE design)
At the start: 60 parts, among them Q1 PMDPB58UPE, U1 MSP430FR5738, U2 SI5351C, U3 PL133-27, U4 SPV1050

Commit message: update hardware design documentation
Parts:
- removed C13, C17: DNP (320p), rcl:C-EUC0402
- removed C14, C18: DNP (400p), rcl:C-EUC0402
- removed C16, C19: DNP (200p), rcl:C-EUC0402
- removed R15, R16: 0, rcl:R-EU_R0201
- added U5: SPV1040, spv1040:SPV1040
- C1: value 100n -> 1u; device rcl:C-EUC0402 -> rcl:C-EUC0603; PARTNO 81-GRM155R71C104KA88 -> (none)
- C2: value 47u -> 10u; device rcl:C-EUC0805 -> rcl:C-EUC0603; PARTNO 81-GRM21BR60J476ME5L -> (none)
- C8: value 4u7 -> 10u; device rcl:C-EUC0603K -> rcl:C-EUC0603; PARTNO 810-C1608X5R1C475KAC -> (none)
- C9: value 10n -> 100n; PARTNO 81-GRM155R71H103MA8D -> (none)
- L1: value 22u -> 10u
- R10: value 8M2 -> 4R7; PARTNO 603-RC0402FR-078M2L -> 603-RC0402FR-07100KL
- R14: value 0 -> 4R7; device rcl:R-EU_R0201 -> rcl:R-EU_R0402; BOM EXCLUDE -> (none); PARTNO (none) -> 603-RC0402FR-07100KL
- R5: value 6M8 -> 1M; PARTNO 603-RC0402FR-076M8L -> (none)
- R6: value 1M5 -> 100k; PARTNO 603-RC0402FR-071M5L -> (none)
- R7: value 2M7 -> 384k; PARTNO 603-RC0402FR-072M7L -> (none)
- R9: value 3M3 -> 1k; PARTNO 603-RC0402FR-073M3L -> (none)
- U4: value SPV1050 -> MIC5304; device SPV1050:SPV1050 -> v-reg-micrel:MIC5219XX; PARTNO 511-SPV1050TTR -> (none)
Connections:
- removed net N$10: L1.2, U4.IN_LV
- removed net N$13: R10.1, R9.2, U4.MPP_SET
- removed net N$14: C9.1, U4.MPP_REF
- removed net PGND: U4.PGND
- new net N$1: Q1G$1.D, R10.2
- new net N$20: R5.1, R7.2, U5.VCTRL
- new net VBAT: C8.1, R5.2, R6.2, R8.1, U4.IN, U5.VOUT, UC1.+
- net +3V3: now also U4.OUT; no longer R15.1, R15.2, R16.1, R16.2, U4.LDO2
- net +3V3_GPS: now also R14.1; no longer Q1G$2.D
- net +3V3_SI: now also R10.1; no longer Q1G$1.D
- net C33: no longer C13.2
- net GND: now also C9.1, R7.1, U5.GND, U5.ICTRL+, U5.ICTRL-; no longer C13.1, C14.1, C16.1, C17.2, C18.2, C19.2, C9.2, R10.2, R7.2, U4.EXP, U4.IN_HV, U4.LDO1_EN, U4.L_HV
- net N$12: no longer C17.1
- net N$15: no longer C18.1
- net N$16: no longer C19.1
- net N$3: no longer C14.2
- net N$4: now also Q1G$2.D; no longer R14.1, R8.1, U4.BATT, U4.LDO2_EN, UC1.+
- net N$5: no longer C16.2
- net N$6: now also U4.EN; no longer R5.2, U4.UVP
- net N$7: now also L1.1, U5.LX; no longer R6.2, R7.1, U4.EOC
- net N$8: now also C9.2, R9.1, U5.MPP_SET; no longer C2.1, R5.1, U4.STORE
- net VSOL_IN: now also C2.1, L1.2, R9.2, U5.XSHUT; no longer C8.1, L1.1, R9.1, U4.CONF, U4.MPP
Other:
- note added: "Symbol of Q1 has gates swapped, patched in software."
- note added: "uTrakHF v1.1 High Altitude Balloon Tracker"
- note added: "uTrakRF v1.1 High Altitude Balloon Tracker"
- note removed: "uTrakHF v1.0 High Altitude Balloon Tracker"
- note removed: "uTrakRF v1.0 High Altitude Balloon Tracker"
- moved on the sheet: C1, C2, C8, C9, L1, Q1G$1, Q1G$2, R10, R11, R14, R3, R4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
